Commit message: Calibrated D435 Cameras.

File: husky_custom_description/urdf/custom_description.urdf.xacro (robot description, xacro)
@@ -26,23 +26,80 @@
   <xacro:arg name="kinect_enabled" default="false" />
   <xacro:include filename="$(find husky_description)/urdf/husky.urdf.xacro" />
-  <xacro:husky_robot />
-  <!-- Insert customization below, sample provided: -->
-  <link name="bowler_link">
+  <xacro:include filename="$(find realsense2_description)/urdf/1_d435.urdf.xacro" />
+  <xacro:include filename="$(find realsense2_description)/urdf/2_d435.urdf.xacro" />
+  <xacro:include filename="$(find realsense2_description)/urdf/3_d435.urdf.xacro" />
+  <!-- <xacro:husky_robot /> -->
+  <!-- Insert customization below, sample provided:
+  <link name="front_camera_mount_link">
     <visual>
       <geometry>
-        <mesh filename="package://husky_custom_description/meshes/red_bowler.dae" />
+        <mesh filename="package://husky_custom_description/meshes/Front_Camera_Assembly.stl" />
       </geometry>
     </visual>
     <collision>
-      <origin xyz="0 0 0.07" rpy="0 0 0" />
+      <origin xyz="0 0 0" rpy="0 0 0" />
       <geometry>
-        <box size="0.32 0.25 0.14" rpy="0 0 0"/>
+        <box size="0.127 0.1016 0.0508" rpy="0 0 0"/>
       </geometry>
     </collision>
   </link>
-  <joint name="bowler_joint" type="fixed">
-    <parent link="top_plate_link" />
-    <child link="bowler_link" />
-    <origin xyz="0.1 -0.1 0" rpy="0 0 0.5" />
+    <joint name="front_camera_mount_joint" type="fixed">
+    <parent link="top_plate_front_link" />
+    <child link="front_camera_mount_link" />
+    <origin xyz="-0.033 -0.063075 -0.00675" rpy="-1.5708 0 1.5708" />
   </joint>
+  <sensor_d435_1 parent="top_plate_camera_mount_link">
+    <origin xyz="0.06289 0.05 0.01585" rpy="3.1415 1.5708 1.5708"/>
+  </sensor_d435_1>
+  -->
+ <link name="top_plate_camera_mount_link">
+    <visual>
+      <geometry>
+        <mesh filename="package://husky_custom_description/meshes/Husky_Top_Plate_with_Cameras_Assembly.stl" />
+      </geometry>
+    </visual>
+    <collision>
+      <origin xyz="0 0 0" rpy="0 0 0" />
+      <geometry>
+        <box size="0.127 0.1016 0.0508" rpy="0 0 0"/>
+      </geometry>
+    </collision>
+  </link>
+   <sensor_d435_1 parent="top_plate_camera_mount_link">
+    <origin xyz="0.117 0.339 0.453" rpy="-1.5708 2.2064 0"/>
+  </sensor_d435_1>
+  <sensor_d435_2 parent="top_plate_camera_mount_link">
+    <origin xyz="0.312 0.337 0.435" rpy="0 1.5708 1.5708"/>
+  </sensor_d435_2>
+  <sensor_d435_3 parent="top_plate_camera_mount_link">
+    <origin xyz="0.508 0.338 0.454" rpy="-1.5708 0.8721 0"/>
+  </sensor_d435_3>
+  <joint name="top_plate_camera_mount_joint" type="fixed">
+    <parent link="top_plate_front_link" />
+    <child link="top_plate_camera_mount_link" />
+    <origin xyz="0.412 0.3115 -0.39326" rpy="-1.5708 3.1415 1.5708" />
+  </joint>
+<!--
+  <joint name="right_camera_mount_joint" type="fixed">
+    <parent link="top_plate_front_link" />
+    <child link="front_camera_mount_link" />
+    <origin xyz="-0.033 -0.063075 -0.00675" rpy="-1.5708 0 1.5708" />
+  </joint>
+  <joint name="left_camera_mount_joint" type="fixed">
+    <parent link="top_plate_front_link" />
+    <child link="front_camera_mount_link" />
+    <origin xyz="-0.033 -0.063075 -0.00675" rpy="-1.5708 0 1.5708" />
+  </joint>
+  <sensor_d435_2 parent="left_side_camera_mount_link">
+    <origin xyz="0.06289 0.05 0.01585" rpy="3.1415 1.5708 1.5708"/>
+  </sensor_d435_2>
+  <sensor_d435_3 parent="right_side_camera_mount_link">
+    <origin xyz="0.06289 0.05 0.01585" rpy="3.1415 1.5708 1.5708"/>
+  </sensor_d435_3>
+  <joint name="front_D435_camera_joint" type="fixed">
+    <parent link="front_camera_mount_link" />
+    <child link="camera2_link" />
+    <origin xyz="0 0 0" rpy="0 3.1415 3.1415" />
+  </joint>
+ -->
 </robot>

Commit message: Modified custom description.

File: husky_custom_description/urdf/custom_description.urdf.xacro (robot description, xacro)
@@ -29,10 +29,10 @@
   <xacro:include filename="$(find realsense2_description)/urdf/2_d435.urdf.xacro" />
   <xacro:include filename="$(find realsense2_description)/urdf/3_d435.urdf.xacro" />
-  <!-- <xacro:husky_robot /> -->
-  <!-- Insert customization below, sample provided:
-  <link name="front_camera_mount_link">
+  <xacro:include filename="$(find realsense2_description)/urdf/4_d435.urdf.xacro" />
+  <xacro:include filename="$(find husky_ur_description)/urdf/husky_ur5_e_description.urdf.xacro"/>
+ <link name="top_plate_ur5_mount_link">
     <visual>
       <geometry>
-        <mesh filename="package://husky_custom_description/meshes/Front_Camera_Assembly.stl" />
+        <mesh filename="package://husky_custom_description/meshes/Husky_End_Effector.stl" />
       </geometry>
     </visual>
@@ -44,14 +44,5 @@
     </collision>
   </link>
-    <joint name="front_camera_mount_joint" type="fixed">
-    <parent link="top_plate_front_link" />
-    <child link="front_camera_mount_link" />
-    <origin xyz="-0.033 -0.063075 -0.00675" rpy="-1.5708 0 1.5708" />
-  </joint>
-  <sensor_d435_1 parent="top_plate_camera_mount_link">
-    <origin xyz="0.06289 0.05 0.01585" rpy="3.1415 1.5708 1.5708"/>
-  </sensor_d435_1>
-  -->
- <link name="top_plate_camera_mount_link">
+   <link name="top_plate_camera_mount_link">
     <visual>
       <geometry>
@@ -66,5 +57,5 @@
     </collision>
   </link>
-   <sensor_d435_1 parent="top_plate_camera_mount_link">
+  <sensor_d435_1 parent="top_plate_camera_mount_link">
     <origin xyz="0.117 0.339 0.453" rpy="-1.5708 2.2064 0"/>
   </sensor_d435_1>
@@ -75,4 +66,7 @@
     <origin xyz="0.508 0.338 0.454" rpy="-1.5708 0.8721 0"/>
   </sensor_d435_3>
+  <sensor_d435_4 parent="top_plate_ur5_mount_link">
+    <origin xyz="0.27 0.105 0.165" rpy="-1.5708 3.1415 1.5708"/>
+  </sensor_d435_4>
   <joint name="top_plate_camera_mount_joint" type="fixed">
     <parent link="top_plate_front_link" />
@@ -80,26 +74,8 @@
     <origin xyz="0.412 0.3115 -0.39326" rpy="-1.5708 3.1415 1.5708" />
   </joint>
-<!--
-  <joint name="right_camera_mount_joint" type="fixed">
-    <parent link="top_plate_front_link" />
-    <child link="front_camera_mount_link" />
-    <origin xyz="-0.033 -0.063075 -0.00675" rpy="-1.5708 0 1.5708" />
+   <joint name="top_plate_ur5_mount_joint" type="fixed">
+    <parent link="ur_arm_wrist_3_link" />
+    <child link="top_plate_ur5_mount_link" />
+    <origin xyz="0.165 0.215 0.122" rpy="0 1.5708 3.1415" />
   </joint>
-  <joint name="left_camera_mount_joint" type="fixed">
-    <parent link="top_plate_front_link" />
-    <child link="front_camera_mount_link" />
-    <origin xyz="-0.033 -0.063075 -0.00675" rpy="-1.5708 0 1.5708" />
-  </joint>
-  <sensor_d435_2 parent="left_side_camera_mount_link">
-    <origin xyz="0.06289 0.05 0.01585" rpy="3.1415 1.5708 1.5708"/>
-  </sensor_d435_2>
-  <sensor_d435_3 parent="right_side_camera_mount_link">
-    <origin xyz="0.06289 0.05 0.01585" rpy="3.1415 1.5708 1.5708"/>
-  </sensor_d435_3>
-  <joint name="front_D435_camera_joint" type="fixed">
-    <parent link="front_camera_mount_link" />
-    <child link="camera2_link" />
-    <origin xyz="0 0 0" rpy="0 3.1415 3.1415" />
-  </joint>
- -->
 </robot>

Commit message: Added transforms for imu.

File: husky_custom_description/urdf/custom_description.urdf.xacro (robot description, xacro)
@@ -57,4 +57,28 @@
     </collision>
   </link>
+  <link name="gx5_link">
+    <collision>
+      <origin xyz="0 0 0" rpy="0 0 0" />
+      <geometry>
+        <box size="0.06 0.025 0.01" rpy="0 0 0"/>
+      </geometry>
+    </collision>
+  </link>
+  <link name="wgs84_odom_link">
+    <collision>
+      <origin xyz="0 0 0" rpy="0 0 0" />
+      <geometry>
+        <box size="0.06 0.025 0.01" rpy="0 0 0"/>
+      </geometry>
+    </collision>
+  </link>
+  <link name="navsat_link">
+    <collision>
+      <origin xyz="0 0 0" rpy="0 0 0" />
+      <geometry>
+        <box size="0.035 0.035 0.015" rpy="0 0 0"/>
+      </geometry>
+    </collision>
+  </link>
   <sensor_d435_1 parent="top_plate_camera_mount_link">
     <origin xyz="0.117 0.339 0.453" rpy="-1.5708 2.2064 0"/>
@@ -74,8 +98,24 @@
     <origin xyz="0.412 0.3115 -0.39326" rpy="-1.5708 3.1415 1.5708" />
   </joint>
-   <joint name="top_plate_ur5_mount_joint" type="fixed">
+  <joint name="top_plate_ur5_mount_joint" type="fixed">
     <parent link="ur_arm_wrist_3_link" />
     <child link="top_plate_ur5_mount_link" />
     <origin xyz="0.165 0.215 0.122" rpy="0 1.5708 3.1415" />
   </joint>
+  <joint name="microstrain_gx5_imu_joint" type="fixed">
+    <parent link="top_plate_link" />
+    <child link="gx5_link" />
+    <origin xyz="-0.09 0.0 -0.07" rpy="3.1415 0 3.1415" />
+    <!--origin xyz="0.0 0.0 0.0" rpy="0 0 0" /-->
+  </joint>
+  <joint name="fused_gps_imu_joint" type="fixed">
+    <parent link="gx5_link" />
+    <child link="wgs84_odom_link" />
+    <origin xyz="0.0 0.0 0.0" rpy=" 0 0 0" />
+  </joint>
+  <joint name="gps_joint" type="fixed">
+    <parent link="top_plate_rear_link" />
+    <child link="navsat_link" />
+    <origin xyz="0.0 0.0 0.27" rpy="0 0 0" />
+  </joint>
 </robot>
